File: REV18/KiCAD/Project/flatlight_rev18/eside_rev18A/eside_rev18.kicad_pcb (KiCad board)
At the start: 2 copper layers, 100 x 60 mm, 49 parts, among them J1 USB_B_Micro, J2 Conn_PROG, J3 Conn_01x04, Q1 DMC1016UPD, SW1 BTN_PWR, SW2 BTN_DIG1, SW3 BTN_DIG2, U1 MCP73831-2x3DFN8, U2 LSM6DS3, U3 ATmega328-MU

Commit message: updated kiCAD
Parts:
- TP1, TP2: footprint lt_foots:TESTPOINT_0.6mm -> TestPoint:TestPoint_Pad_1.0x1.0mm; moved to F.Cu
- moved TP1 2.06 mm to (69.7, 98.1), turned to 90 degrees
- moved TP2 1.90 mm to (69.8, 101.7), turned to 90 degrees
- moved R7 0.10 mm to (147.1, 84.2)
Routing:
- net TX: track 4.45 -> 6.21 mm, vias 0 -> 1
Changed lines of the file:
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@@
     (thickness 1.6)
     (drawings 8)
-    (tracks 438)
+    (tracks 439)
     (zones 0)
     (modules 49)
@@
     (47 F.CrtYd user)
     (48 B.Fab user)
-    (49 F.Fab user)
+    (49 F.Fab user hide)
   )
   (setup
@@
     (add_net MISO)
     (add_net MOSI)
+    (add_net "Net-(BT1-Pad1)")
+    (add_net "Net-(BT1-Pad2)")
+    (add_net "Net-(BT1-Pad3)")
+    (add_net "Net-(BT1-Pad4)")
     (add_net "Net-(C3-Pad1)")
     (add_net "Net-(C5-Pad2)")
     (add_net "Net-(C6-Pad1)")
     (add_net "Net-(D1-Pad2)")
+    (add_net "Net-(D1-Pad3)")
     (add_net "Net-(D1-Pad4)")
     (add_net "Net-(D2-Pad2)")
     (add_net "Net-(D2-Pad3)")
+    (add_net "Net-(D3-Pad2)")
+    (add_net "Net-(D3-Pad3)")
+    (add_net "Net-(J1-Pad2)")
+    (add_net "Net-(J1-Pad3)")
+    (add_net "Net-(J1-Pad4)")
     (add_net "Net-(Q1-Pad2)")
     (add_net "Net-(Q1-Pad4)")
@@
     (add_net "Net-(R8-Pad2)")
     (add_net "Net-(R9-Pad2)")
+    (add_net "Net-(U1-Pad7)")
+    (add_net "Net-(U2-Pad10)")
+    (add_net "Net-(U2-Pad11)")
+    (add_net "Net-(U2-Pad12)")
+    (add_net "Net-(U3-Pad11)")
+    (add_net "Net-(U3-Pad12)")
+    (add_net "Net-(U3-Pad19)")
+    (add_net "Net-(U3-Pad2)")
+    (add_net "Net-(U3-Pad22)")
+    (add_net "Net-(U3-Pad30)")
+    (add_net "Net-(U3-Pad7)")
+    (add_net "Net-(U3-Pad8)")
     (add_net OC1A)
     (add_net OC1B)
@@
     (add_net VCC)
   )
+  (module TestPoint:TestPoint_Pad_1.0x1.0mm (layer F.Cu)
+    (at 69.8 101.7 90)
+    (descr "SMD rectangular pad as test Point, square 1.0mm side length")
+    (tags "test point SMD pad rectangle square")
+    (attr virtual)
+    (fp_text reference TP2 (at 0 -1.448 -90) (layer F.SilkS)
+      (effects (font (size 1 1) (thickness 0.15)))
+    )
+    (fp_text value TestPoint (at 0 1.55 -90) (layer F.Fab)
+      (effects (font (size 1 1) (thickness 0.15)))
+    )
+    (fp_line (start 1 1) (end -1 1) (layer F.CrtYd) (width 0.05))
+    (fp_line (start 1 1) (end 1 -1) (layer F.CrtYd) (width 0.05))
+    (fp_line (start -1 -1) (end -1 1) (layer F.CrtYd) (width 0.05))
+    (fp_line (start -1 -1) (end 1 -1) (layer F.CrtYd) (width 0.05))
+    (fp_line (start -0.7 0.7) (end -0.7 -0.7) (layer F.SilkS) (width 0.12))
+    (fp_line (start 0.7 0.7) (end -0.7 0.7) (layer F.SilkS) (width 0.12))
+    (fp_line (start 0.7 -0.7) (end 0.7 0.7) (layer F.SilkS) (width 0.12))
+    (fp_line (start -0.7 -0.7) (end 0.7 -0.7) (layer F.SilkS) (width 0.12))
+    (fp_text user %R (at 0 -1.45 -90) (layer F.Fab)
+      (effects (font (size 1 1) (thickness 0.15)))
+    )
+    (pad 1 smd rect (at 0 0 90) (size 1 1) (layers F.Cu F.Mask)
+      (net 30 TX))
+  )
+  (module TestPoint:TestPoint_Pad_1.0x1.0mm (layer F.Cu)
+    (at 69.7 98.1 90)
+    (descr "SMD rectangular pad as test Point, square 1.0mm side length")
+    (tags "test point SMD pad rectangle square")
+    (attr virtual)
+    (fp_text reference TP1 (at 0 -1.448 -90) (layer F.SilkS)
+      (effects (font (size 1 1) (thickness 0.15)))
+    )
+    (fp_text value TestPoint (at 0 1.55 -90) (layer F.Fab)
+      (effects (font (size 1 1) (thickness 0.15)))
+    )
+    (fp_line (start 1 1) (end -1 1) (layer F.CrtYd) (width 0.05))
+    (fp_line (start 1 1) (end 1 -1) (layer F.CrtYd) (width 0.05))
+    (fp_line (start -1 -1) (end -1 1) (layer F.CrtYd) (width 0.05))
+    (fp_line (start -1 -1) (end 1 -1) (layer F.CrtYd) (width 0.05))
+    (fp_line (start -0.7 0.7) (end -0.7 -0.7) (layer F.SilkS) (width 0.12))
+    (fp_line (start 0.7 0.7) (end -0.7 0.7) (layer F.SilkS) (width 0.12))
+    (fp_line (start 0.7 -0.7) (end 0.7 0.7) (layer F.SilkS) (width 0.12))
+    (fp_line (start -0.7 -0.7) (end 0.7 -0.7) (layer F.SilkS) (width 0.12))
+    (fp_text user %R (at 0 -1.45 -90) (layer F.Fab)
+      (effects (font (size 1 1) (thickness 0.15)))
+    )
+    (pad 1 smd rect (at 0 0 90) (size 1 1) (layers F.Cu F.Mask)
+      (net 2 GND))
+  )
   (module lt_foots:logo_heart3 (layer F.Cu)
     (at 139.5 58.7)
@@
   )
   (module Resistor_SMD:R_0603_1608Metric (layer B.Cu)
-    (at 147 84.2 270)
+    (at 147.1 84.2 270)
     (descr "Resistor SMD 0603 (1608 Metric), square (rectangular) end terminal, IPC_7351 nominal, (Body size source: http://www.tortai-tech.com/upload/download/2011102023233369053.pdf), generated with kicad-footprint-generator")
     (tags resistor)
@@
     )
   )
-  (module lt_foots:TESTPOINT_0.6mm (layer B.Cu)
-    (at 69.2 99.9 270)
-    (fp_text reference TP2 (at 1.9 -1 180) (layer B.SilkS) hide
-      (effects (font (size 1 1) (thickness 0.15)) (justify mirror))
-    )
-    (fp_text value TestPoint (at -0.5 -0.2 90) (layer B.Fab)
-      (effects (font (size 1 1) (thickness 0.15)) (justify mirror))
-    )
-    (pad 1 thru_hole circle (at 0 0 270) (size 0.6 0.6) (drill 0.3) (layers *.Cu *.Mask)
-      (net 30 TX))
-  )
-  (module lt_foots:TESTPOINT_0.6mm (layer B.Cu)
-    (at 70.7 99.9 270)
-    (fp_text reference TP1 (at 2.2 0 180) (layer B.SilkS) hide
-      (effects (font (size 1 1) (thickness 0.15)) (justify mirror))
-    )
-    (fp_text value TestPoint (at -0.4 -0.1 90) (layer B.Fab)
-      (effects (font (size 1 1) (thickness 0.15)) (justify mirror))
-    )
-    (pad 1 thru_hole circle (at 0 0 270) (size 0.6 0.6) (drill 0.3) (layers *.Cu *.Mask)
-      (net 2 GND))
-  )
   (module Connector_USB:USB_Micro-B_Wuerth_629105150521 (layer B.Cu)
     (at 139.1 105.8 180)
@@
   (segment (start 145.35 64.4) (end 145.35 65.8) (width 1) (layer B.Cu) (net 1))
   (segment (start 145.1 66) (end 143.5 66) (width 0.6) (layer B.Cu) (net 1))
-  (segment (start 122.4 98.535) (end 125 98.535) (width 0.6) (layer B.Cu) (net 1))
+  (segment (start 122.5 98.535) (end 125.1 98.535) (width 1) (layer B.Cu) (net 1))
   (segment (start 124.3 101.5) (end 123.2875 101.5) (width 0.6) (layer B.Cu) (net 1))
   (segment (start 124.7 99) (end 124.7 101.1) (width 0.6) (layer B.Cu) (net 1))
@@
   (segment (start 144.65 76.85) (end 144.4 77.1) (width 0.3) (layer B.Cu) (net 2))
   (segment (start 145.85 76.85) (end 144.65 76.85) (width 0.3) (layer B.Cu) (net 2))
-  (segment (start 146.525 76.85) (end 146.7 77.025) (width 0.3) (layer B.Cu) (net 2))
-  (segment (start 145.85 76.85) (end 146.525 76.85) (width 0.3) (layer B.Cu) (net 2))
   (segment (start 101.2625 97.15) (end 102.25 97.15) (width 0.2) (layer B.Cu) (net 2))
   (segment (start 101.2625 97.65) (end 102.15 97.65) (width 0.2) (layer B.Cu) (net 2))
@@
   (via (at 128.8 93.1) (size 0.6) (drill 0.3) (layers F.Cu B.Cu) (net 2))
   (via (at 128.8 92.1) (size 0.6) (drill 0.3) (layers F.Cu B.Cu) (net 2))
+  (segment (start 146.55 76.85) (end 146.6 76.9) (width 0.3) (layer B.Cu) (net 2))
+  (segment (start 145.85 76.85) (end 146.55 76.85) (width 0.3) (layer B.Cu) (net 2))
   (segment (start 140.6 103.9) (end 140.6 102.375) (width 0.8) (layer B.Cu) (net 3))
   (segment (start 140.4 102.5) (end 140.4 98.9) (width 1) (layer B.Cu) (net 3))
@@
   (segment (start 98.8375 98.15) (end 96.55 98.15) (width 0.2) (layer B.Cu) (net 29))
   (segment (start 96.55 98.15) (end 96.3 98.4) (width 0.2) (layer B.Cu) (net 29))
-  (segment (start 68 99.9) (end 69.2 99.9) (width 0.4) (layer B.Cu) (net 30))
-  (segment (start 64.9375 100.35) (end 67.55 100.35) (width 0.2) (layer B.Cu) (net 30))
-  (segment (start 67.55 100.35) (end 68 99.9) (width 0.2) (layer B.Cu) (net 30))
+  (segment (start 64.9375 100.35) (end 69.8 100.35) (width 0.2) (layer B.Cu) (net 30))
+  (segment (start 69.8 100.35) (end 69.8 100.35) (width 0.2) (layer B.Cu) (net 30))
+  (via (at 69.8 100.35) (size 0.6) (drill 0.3) (layers F.Cu B.Cu) (net 30))
+  (segment (start 69.8 101.7) (end 69.8 100.35) (width 0.6) (layer F.Cu) (net 30))
   (segment (start 123.4375 103.45) (end 123.2875 103.3) (width 0.2) (layer B.Cu) (net 31))
   (segment (start 123.4375 105.1) (end 123.4375 103.45) (width 0.6) (layer B.Cu) (net 31))
