File: REV18/KiCAD/Project/flatlight_rev18/eside_rev18A/eside_rev18.sch (KiCad schematic (older format))
At the start: 49 parts, among them J1 USB_B_Micro, J2 Conn_PROG, J3 Conn_01x04, Q1 DMC1016UPD, SW1 BTN_PWR, SW2 BTN_DIG1, SW3 BTN_DIG2, U1 MCP73831-2x3DFN8, U2 LSM6DS3, U3 ATmega328-MU

Commit message: updated kiCAD
Parts:
- TP1, TP2: footprint lt_foots:TESTPOINT_0.6mm -> TestPoint:TestPoint_Pad_1.0x1.0mm
Changed lines of the file:
@@
 F 0 "TP1" V 6559 3858 50  0000 L CNN
 F 1 "TestPoint" V 6650 3858 50  0000 L CNN
-F 2 "lt_foots:TESTPOINT_0.6mm" H 6805 3670 50  0001 C CNN
+F 2 "TestPoint:TestPoint_Pad_1.0x1.0mm" H 6805 3670 50  0001 C CNN
 F 3 "~" H 6805 3670 50  0001 C CNN
 	1    6605 3670
@@
 F 0 "TP2" V 6580 4300 50  0000 R CNN
 F 1 "TestPoint" V 6660 4515 50  0000 R CNN
-F 2 "lt_foots:TESTPOINT_0.6mm" H 6815 3980 50  0001 C CNN
+F 2 "TestPoint:TestPoint_Pad_1.0x1.0mm" H 6815 3980 50  0001 C CNN
 F 3 "~" H 6815 3980 50  0001 C CNN
 	1    6615 3980
