File: REV18/KiCAD/Project/flatlight_rev18/ledside_rev18A/ledside_rev18A.kicad_pcb (KiCad board)
At the start: 2 copper layers, 100 x 60 mm, 38 parts, among them J1 Conn_01x04, Q1 DMN2022-UFDF7, Q2 DMN2022-UFDF7

Commit message: updated kiCAD
Routing:
- net LED_NTC2: vias 2 -> 1
- net GND: vias 39 -> 41
Changed lines of the file:
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@@
     (thickness 1.6)
     (drawings 8)
-    (tracks 147)
+    (tracks 148)
     (zones 0)
     (modules 38)
@@
   (segment (start 110.950112 42.651504) (end 111.000112 42.601504) (width 0.2) (layer F.Cu) (net 2))
   (segment (start 110.050112 42.651504) (end 110.950112 42.651504) (width 0.2) (layer F.Cu) (net 2))
-  (via (at 107.5 48.45) (size 0.6) (drill 0.3) (layers F.Cu B.Cu) (net 2))
-  (via (at 107.5 53.65) (size 0.6) (drill 0.3) (layers F.Cu B.Cu) (net 2))
-  (via (at 107.5 50.15) (size 0.6) (drill 0.3) (layers F.Cu B.Cu) (net 2))
-  (via (at 107.5 51.9) (size 0.6) (drill 0.3) (layers F.Cu B.Cu) (net 2))
   (via (at 21.5 55) (size 0.6) (drill 0.3) (layers F.Cu B.Cu) (net 2))
   (via (at 21.5 60) (size 0.6) (drill 0.3) (layers F.Cu B.Cu) (net 2))
@@
   (via (at 118.5 45) (size 0.6) (drill 0.3) (layers F.Cu B.Cu) (net 2))
   (via (at 118.5 42.5) (size 0.6) (drill 0.3) (layers F.Cu B.Cu) (net 2))
+  (via (at 109.2 49) (size 0.6) (drill 0.3) (layers F.Cu B.Cu) (net 2))
+  (via (at 109.2 51) (size 0.6) (drill 0.3) (layers F.Cu B.Cu) (net 2))
+  (via (at 109.2 50) (size 0.6) (drill 0.3) (layers F.Cu B.Cu) (net 2))
+  (via (at 108.2 49) (size 0.6) (drill 0.3) (layers F.Cu B.Cu) (net 2))
+  (via (at 108.2 50) (size 0.6) (drill 0.3) (layers F.Cu B.Cu) (net 2))
+  (via (at 108.2 51) (size 0.6) (drill 0.3) (layers F.Cu B.Cu) (net 2))
   (segment (start 70 77.3) (end 70 44.8) (width 5) (layer B.Cu) (net 3))
   (via (at 75 78.5) (size 0.6) (drill 0.3) (layers F.Cu B.Cu) (net 3))
@@
   (segment (start 109.750112 41.951504) (end 110.050112 41.651504) (width 0.2) (layer F.Cu) (net 8))
   (segment (start 109.100112 41.951504) (end 109.750112 41.951504) (width 0.2) (layer F.Cu) (net 8))
-  (via (at 107.5 46.7) (size 0.6) (drill 0.3) (layers F.Cu B.Cu) (net 9))
   (segment (start 107.3 25.375) (end 107.3 27.8) (width 0.6) (layer F.Cu) (net 9))
   (segment (start 118.55 47) (end 115.675 47) (width 0.6) (layer F.Cu) (net 9))
